Commit message: removed typos

File: jazzy_ws/src/grr_description/urdf/control/drive.xacro (robot description, xacro)
@@ -1,4 +1,6 @@
 <?xml version="1.0"?>
 <robot xmlns:xacro="http://www.ros.org/wiki/xacro">
+  <xacro:arg name="hardware_interface" default="CanInterface" />
+  <xacro:property name="hardware_interface_value" value="$(arg hardware_interface)" />
   <ros2_control name="gregg" type="system">
     <hardware>
@@ -11,5 +13,4 @@
         <param name="controlled_joints">front_right_mecanum_joint, front_left_mecanum_joint, rear_right_mecanum_joint, rear_left_mecanum_joint</param>
       </xacro:if>
-    </hardware>
     </hardware>
     <joint name="front_right_mecanum_joint">
